File: keyfrick.kicad_pcb (KiCad board)
At the start: 2 copper layers, 96 x 34 mm, 13 parts, among them SW1 SW_Push, SW2 SW_Push, SW3 SW_Push, SW4 SW_Push, U1 XIAO-RP2040-DIP

Commit message: routed pcb traces
Routing:
- net GND: track 0.00 -> 101.6 mm
- net d1: track 0.00 -> 89.6 mm
- net sw1: track 0.00 -> 77.6 mm
- net d2: track 0.00 -> 71.1 mm
- net sw2: track 0.00 -> 55.4 mm
- net d3: track 0.00 -> 50.4 mm
- net sw3: track 0.00 -> 33.1 mm
- net d4: track 0.00 -> 32.3 mm
- net sw4: track 0.00 -> 10.9 mm
- net Net-(D2-PadA): track 0.00 -> 5.69 mm
- net Net-(D4-PadA): track 0.00 -> 5.69 mm
- net Net-(D3-PadA): track 0.00 -> 5.69 mm
- net Net-(D1-PadA): track 0.00 -> 5.69 mm
